File: badgeInventor.kicad_pcb (KiCad board)
At the start: 2 copper layers, 81.6 x 61.3 mm, 36 parts, among them P1 AUTO-PROGRAM JUMPER, P2 CONN_01X10, P22 CONN_01X10, P23 CONN_01X10, P3 LiPo, P5 OLED_I2C, P6 USB Serial, SW1 RESET, SW2 SW_PUSH, U1 SPX1117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

Commit message: Agregado logos y para colgar
Parts:
- removed the G*** at (139.4, 119.4)
- added G***: LOGO, theinventorhouse:electronic_cats_logo_8x6, B.Cu at (152.1, 141.7)
- added G***: LOGO, theinventorhouse:intel_logo, B.Cu at (140.4, 141.8)
- LED1: value MADW__WS2812B -> WS2812B
- P1: value AUTO-PROGRAM JUMPER -> PROG_JUMP
Other:
- outline, holes or cut-outs redrawn
- board text added: "Power by"
- board text removed: "PROG_JUMP"
